File: AND/AND.kicad_pcb (KiCad board)
At the start: 2 copper layers, 10 parts

Commit message: Add files via upload
Other:
- board outline added: 33.7 x 17.8 mm
- board text added: "the spaghetti made of codes"
- board text removed: "the code made of spaghetti"

Commit message: Add files via upload
Parts:
- REF** (x6): moved to B.Cu
Other:
- board size 33.7 x 17.8 mm -> 33.3 x 17.8 mm
- board text added: "the spaghetti made of code"
- board text removed: "the spaghetti made of codes"

Commit message: Add files via upload
Parts:
- removed REF** (x2): Condensor, MiyakeFootprintLib:Condensor
- removed REF** (x2): 946H-1C-24D, MiyakeFootprintLib:946H-1C-24D
- removed REF** (x6): PinHeader_1x01_P2.54mm_Vertical, Connector_PinHeader_2.54mm:PinHeader_1x01_P2.54mm_Vertical
- added C1: C, MiyakeFootprintLib:Condensor, F.Cu at (109.2, 108.6)
- added C2: C, MiyakeFootprintLib:Condensor, F.Cu at (127.0, 104.8)
- added J1: Conn_01x01, Connector_PinHeader_2.54mm:PinHeader_1x01_P2.54mm_Vertical, B.Cu at (106.7, 102.2)
- added J2: Conn_01x01, Connector_PinHeader_2.54mm:PinHeader_1x01_P2.54mm_Vertical, B.Cu at (109.2, 102.2)
- added J3: Conn_01x01, Connector_PinHeader_2.54mm:PinHeader_1x01_P2.54mm_Vertical, B.Cu at (121.9, 102.2)
- added J4: Conn_01x01, Connector_PinHeader_2.54mm:PinHeader_1x01_P2.54mm_Vertical, B.Cu at (124.9, 102.2)
- added J5: Conn_01x02, Connector_PinHeader_2.54mm:PinHeader_1x02_P2.54mm_Vertical, B.Cu at (109.2, 114.3)
- added SPDT1: 946H-1C-24D, MiyakeFootprintLib:946H-1C-24D, F.Cu at (101.6, 106.8)
- added SPDT2: 946H-1C-24D, MiyakeFootprintLib:946H-1C-24D, F.Cu at (116.8, 106.8)
Routing:
- net (no net): track 135.6 -> 0.00 mm
- net GND: track 0.00 -> 50.9 mm
- net +24V: track 0.00 -> 31.0 mm
- net Net-(J3-Pad1): track 0.00 -> 26.8 mm
- net Net-(C2-Pad2): track 0.00 -> 19.9 mm
- net Net-(C1-Pad1): track 0.00 -> 10.3 mm
- removed copper zone on B.Cu, net GND
- removed copper zone on F.Cu, net GND
Other:
- board size 33.3 x 17.8 mm -> 33.7 x 17.8 mm
- board text added: "I0"
- board text added: "I1"
- board text removed: "C"
- board text removed: "IN"

Commit message: Add files via upload
Parts:
- J5: moved to F.Cu
- moved C2 23.3 mm to (123.4, 127.8)
- moved J4 23.1 mm to (121.9, 125.1)
- moved J1 23.0 mm to (104.1, 125.1)
- moved J2 23.0 mm to (106.7, 125.1)
- moved J3 23.0 mm to (119.4, 125.1)
- moved J5 23.0 mm to (106.7, 137.2), turned to 180 degrees
- moved C1 22.9 mm to (106.7, 131.3)
- moved SPDT1 22.9 mm to (99.1, 129.5)
- moved SPDT2 22.9 mm to (114.3, 129.5)
Routing:
- net GND: track 50.9 -> 53.2 mm
- net Net-(C2-Pad2): track 19.9 -> 18.9 mm
- net Net-(J3-Pad1): track 26.8 -> 27.5 mm
- net +24V: track 31.0 -> 30.4 mm
- added copper zone on B.Cu, net GND
- added copper zone on F.Cu, net GND
Other:
- board size 33.7 x 17.8 mm -> 33 x 17.8 mm
- board text added: "C"

Commit message: Add files via upload
Parts:
- removed J4: Conn_01x01, Connector_PinHeader_2.54mm:PinHeader_1x01_P2.54mm_Vertical
- removed J5: Conn_01x02, Connector_PinHeader_2.54mm:PinHeader_1x02_P2.54mm_Vertical
- J1, J2, J3: value Conn_01x01 -> Conn_01x02; footprint Connector_PinHeader_2.54mm:PinHeader_1x01_P2.54mm_Vertical -> Connector_PinHeader_2.54mm:PinHeader_1x02_P2.54mm_Vertical
- moved J1 53.9 mm to (66.0, 87.0), turned to 270 degrees
- moved SPDT1 53.9 mm to (61.0, 91.4)
- moved SPDT2 53.9 mm to (76.2, 91.4)
- moved C1 53.8 mm to (68.6, 93.3)
- moved C2 52.9 mm to (83.8, 92.7), turned to 180 degrees
- moved J3 52.1 mm to (83.8, 87.0), turned to 90 degrees
- moved J2 47.6 mm to (68.6, 96.5), turned to 180 degrees
Connections:
- J2 pad 1: Net-(C2-Pad2) -> GND
- SPDT1 pad 2: +24V -> Net-(SPDT1-Pad2)
- SPDT2 pad 1: +24V -> Net-(SPDT2-Pad1)
- SPDT2 pad 2: +24V -> Net-(SPDT1-Pad2)
Routing:
- net Net-(SPDT1-Pad2): track 0.00 -> 26.8 mm
- net +24V: track 30.4 -> 5.08 mm
- net Net-(J3-Pad1): track 27.5 -> 18.2 mm
- net Net-(C2-Pad2): track 18.9 -> 15.1 mm
- net GND: track 53.2 -> 50.8 mm
- net Net-(C1-Pad1): track 10.2 -> 11.0 mm
