File: NAND/NAND.kicad_pcb (KiCad board)
At the start: 2 copper layers, 35.6 x 17.8 mm, 10 parts

Commit message: Add files via upload
Parts:
- removed REF** (x2): Condensor, MiyakeFootprintLib:Condensor
- removed REF** (x2): 946H-1C-24D, MiyakeFootprintLib:946H-1C-24D
- removed REF** (x6): PinHeader_1x01_P2.54mm_Vertical, Connector_PinHeader_2.54mm:PinHeader_1x01_P2.54mm_Vertical
- added C1: C, MiyakeFootprintLib:Condensor, F.Cu at (106.7, 54.6)
- added C2: C, MiyakeFootprintLib:Condensor, F.Cu at (121.9, 54.6)
- added J1: Conn_01x02, Connector_PinHeader_2.54mm:PinHeader_1x02_P2.54mm_Vertical, B.Cu at (104.1, 48.9)
- added J2: Conn_01x02, Connector_PinHeader_2.54mm:PinHeader_1x02_P2.54mm_Vertical, B.Cu at (106.7, 58.4)
- added J3: Conn_01x02, Connector_PinHeader_2.54mm:PinHeader_1x02_P2.54mm_Vertical, B.Cu at (121.9, 48.9)
- added SPDT1: 946H-1C-24D, MiyakeFootprintLib:946H-1C-24D, F.Cu at (99.1, 53.3)
- added SPDT2: 946H-1C-24D, MiyakeFootprintLib:946H-1C-24D, F.Cu at (114.3, 53.3)
Routing:
- net (no net): track 110.9 -> 0.00 mm
- net GND: track 0.00 -> 50.9 mm
- net Net-(C2-Pad2): track 0.00 -> 29.1 mm
- net Net-(J3-Pad1): track 0.00 -> 21.8 mm
- net Net-(J1-Pad2): track 0.00 -> 14.9 mm
- net Net-(C1-Pad1): track 0.00 -> 10.7 mm
- net +24V: track 0.00 -> 2.54 mm
Other:
- board size 35.6 x 17.8 mm -> 33 x 17.8 mm
- board text added: "I0"
- board text added: "I1"
- board text removed: "IN"
